File: demo/adder/half-adder.kicad_sch (KiCad schematic)
At the start: 8 parts

Commit message: Component Circuit revise - simplify design - implement full circuit
Parts:
- added LR1, LR2: (no value), symbol component-symbols:redstone-button
- added LR37, LR38, LR40, LR42: (no value), symbol component-symbols:redstone-torch
- added LR39, LR41, LR43, LR44: (no value), symbol component-symbols:redstone-repeater
- renumbered LR61 to LR69, LR62 to LR70, LR63 to LR71, LR64 to LR72, LR65 to LR73, LR66 to LR74, LR67 to LR75, LR68 to LR76
Connections:
- net CARRY: now also LR44.3
- net RESULT: now also LR41.3
- new net: LR42.1, LR43.3
- new net: LR41.2, LR42.2
- new net: LR37.2, LR39.1
- new net: LR39.2, LR40.2
- new net: LR38.1, LR39.3
- new net: LR38.2, LR41.1
- new net: LR1.1, LR40.1, LR43.2
- new net: LR2.1, LR37.1, LR43.1
