File: dev/FalloutProject.kicad_sch (KiCad schematic)
At the start: 65 parts, among them Q1 2N3904, Q2 2N3904, Q3 2N3904, Q4 2N3904, Q5 2N3904, Q6 KPS-3227, SW1 SW_Push, SW2 SW_Push, SW3 SW_Push

Commit message: Add README of demo - "Adder - LogicalRedstone Project Demo"
Parts:
- added LR45: (no value), symbol component-symbols:redstone-block
- added LR46: (no value), symbol component-symbols:redstone-button
- added LR47: (no value), symbol component-symbols:redstone-lamp
- added LR48: (no value), symbol component-symbols:redstone-repeater
- added LR49: (no value), symbol component-symbols:redstone-torch
Other:
- note added: "redstone-block"
- note added: "redstone-button"
- note added: "redstone-lamp"
- note added: "redstone-repeater"
- note added: "redstone-torch"
